Commit message: Fix package name

File: urdf/teraranger_evo.urdf.xacro (robot description, xacro)
@@ -7,5 +7,5 @@
                     <origin xyz="0.0 0.0 0.0" rpy="0 0 0"/>
                     <geometry>
-                        <mesh filename="package://teraranger_tower_evo_description/meshes/teraranger_evo.stl"/>
+                        <mesh filename="package://teraranger_description/meshes/teraranger_evo.stl"/>
                     </geometry>
                     <material name="Yellow">
@@ -61,5 +61,5 @@
                     <origin xyz="0.0 0 0.0" rpy="0 0 0"/>
                     <geometry>
-                        <mesh filename="package://teraranger_tower_evo_description/meshes/teraranger_evo.stl"/>
+                        <mesh filename="package://teraranger_description/meshes/teraranger_evo.stl"/>
                     </geometry>
                     <material name="Yellow"/>

File: urdf/teraranger_evo_tower.urdf (robot description, URDF)
Before this commit: robot teraranger_evo_tower.urdf, 1 links, 0 joints
Links:
- link base_link: geometry collision box size=0.1 0.1 0.1; visual mesh filename=$(find teraranger_description)/meshes/Evo_Tower.stl

File: urdf/teraranger_evo_tower.urdf.xacro (robot description, xacro)
@@ -2,5 +2,5 @@
 <robot name="teraranger_evo_tower" xmlns:xacro="http://www.ros.org/wiki/xacro">
     <xacro:include filename="$(find teraranger_description)/urdf/base_hub.urdf.xacro"/>
-    <xacro:include filename="$(find teraranger_tower_evo_description)/urdf/teraranger_evo.urdf.xacro"/>
+    <xacro:include filename="$(find teraranger_description)/urdf/teraranger_evo.urdf.xacro"/>
     <xacro:macro name="teraranger_evo_tower" params="multi_hub hub_id parent x y z roll pitch yaw">
       <!-- EVO TOWER CONFIG-->

File: urdf/teraranger_multiflex.urdf.xacro (robot description, xacro)
@@ -7,5 +7,5 @@
                     <origin xyz="0.0 0.0 0.0" rpy="0 0 0"/>
                     <geometry>
-                        <mesh filename="package://teraranger_tower_evo_description/meshes/teraranger_multiflex.stl"/>
+                        <mesh filename="package://teraranger_description/meshes/teraranger_multiflex.stl"/>
                     </geometry>
                     <material name="Yellow">
@@ -61,5 +61,5 @@
                     <origin xyz="0.0 0 0.0" rpy="0 0 0"/>
                     <geometry>
-                        <mesh filename="package://teraranger_tower_evo_description/meshes/teraranger_evo.stl"/>
+                        <mesh filename="package://teraranger_description/meshes/teraranger_evo.stl"/>
                     </geometry>
                     <material name="Yellow"/>

Commit message: Update teraranger_evo.urdf.xacro
Add cuboid inertia for Teraranger Evo

File: urdf/teraranger_evo.urdf.xacro (robot description, xacro)
@@ -18,4 +18,16 @@
                 <parent link="base_hub_${hub_id}"/>
                 <child link="hub_${hub_id}_base_range_${id}"/>
+            </joint>
+            <link name="inertial_link_${hub_id}_base_range_joint_${id}">
+              <inertial>
+                  <mass value="0.010"/>
+                  <origin xyz="0 0 0"/>
+                  <inertia ixx="1.2e-6" ixy="0" ixz="0" iyy="1.5e-6" iyz="0" izz="1.2e-6"/>
+              </inertial>
+            </link>
+            <joint name="inertial_joint_${hub_id}" type="fixed">
+              <origin xyz="0.0 0.0 0" rpy="0 0 0" />
+              <parent link="base_hub_${hub_id}"/>
+              <child link="inertial_link_${hub_id}_base_range_joint_${id}"/>
             </joint>
             <gazebo reference="hub_${hub_id}_base_range_${id}">
@@ -71,4 +83,16 @@
                 <child link="base_range_${id}"/>
             </joint>
+            <link name="inertial_link_base_range_joint_${id}">
+              <inertial>
+                  <mass value="0.010"/>
+                  <origin xyz="0 0 0"/>
+                  <inertia ixx="1.2e-6" ixy="0" ixz="0" iyy="1.5e-6" iyz="0" izz="1.2e-6"/>
+              </inertial>
+            </link>
+            <joint name="inertial_joint_${hub_id}" type="fixed">
+              <origin xyz="0.0 0.0 0" rpy="0 0 0" />
+              <parent link="base_hub"/>
+              <child link="inertial_link_base_range_joint_${id}"/>
+            </joint>
             <gazebo reference="base_range_${id}">
                 <material>Gazebo/Yellow</material>
