Commit message: Correct references to old package

File: urdf/teraranger_one.urdf.xacro (robot description, xacro)
@@ -7,5 +7,5 @@
                     <origin xyz="0 0 -0.005" rpy="0 0 0"/>
                     <geometry>
-                        <mesh filename="package://teraranger_tower_description/meshes/trone.dae"/>
+                        <mesh filename="package://teraranger_description/meshes/trone.dae"/>
                     </geometry>
                     <material name="Yellow"/>
@@ -59,5 +59,5 @@
                     <origin xyz="0 0 -0.005" rpy="0 0 0"/>
                     <geometry>
-                        <mesh filename="package://teraranger_tower_description/meshes/trone.dae"/>
+                        <mesh filename="package://teraranger_description/meshes/trone.dae"/>
                     </geometry>
                     <material name="Yellow"/>

File: urdf/teraranger_tower.urdf.xacro (robot description, xacro)
@@ -1,6 +1,6 @@
 <?xml version="1.0"?>
 <robot name="teraranger_tower" xmlns:xacro="http://www.ros.org/wiki/xacro">
-    <xacro:include filename="$(find teraranger_tower_description)/urdf/base_hub.urdf.xacro"/>
-    <xacro:include filename="$(find teraranger_tower_description)/urdf/teraranger_one.urdf.xacro"/>
+    <xacro:include filename="$(find teraranger_description)/urdf/base_hub.urdf.xacro"/>
+    <xacro:include filename="$(find teraranger_description)/urdf/teraranger_one.urdf.xacro"/>
     <xacro:macro name="teraranger_tower" params="multi_hub hub_id parent x y z roll pitch yaw">
         <base_hub multi_hub="${multi_hub}" hub_id='${hub_id}' parent="${parent}" x="${x}" y="${y}" z="${z}" roll="${roll}" pitch="${pitch}" yaw="${yaw}" />

Commit message: Update teraranger_one.urdf.xacro
Add cuboid inertia to TeraRanger One

File: urdf/teraranger_one.urdf.xacro (robot description, xacro)
@@ -16,4 +16,16 @@
                 <parent link="base_hub_${hub_id}"/>
                 <child link="hub_${hub_id}_base_range_${id}"/>
+            </joint>
+            <link name="inertial_link_${hub_id}_base_range_joint_${id}">
+              <inertial>
+                  <mass value="0.010"/>
+                  <origin xyz="0 0 0"/>
+                  <inertia ixx="1.2e-6" ixy="0" ixz="0" iyy="1.5e-6" iyz="0" izz="1.2e-6"/>
+              </inertial>
+            </link>
+            <joint name="inertial_joint_${hub_id}" type="fixed">
+              <origin xyz="0.0 0.0 0" rpy="0 0 0" />
+              <parent link="base_hub_${hub_id}"/>
+              <child link="inertial_link_${hub_id}_base_range_joint_${id}"/>
             </joint>
             <gazebo reference="hub_${hub_id}_base_range_${id}">
@@ -69,4 +81,16 @@
                 <child link="base_range_${id}"/>
             </joint>
+            <link name="inertial_link_base_range_joint_${id}">
+              <inertial>
+                  <mass value="0.010"/>
+                  <origin xyz="0 0 0"/>
+                  <inertia ixx="1.2e-6" ixy="0" ixz="0" iyy="1.5e-6" iyz="0" izz="1.2e-6"/>
+              </inertial>
+            </link>
+            <joint name="inertial_joint_${hub_id}" type="fixed">
+              <origin xyz="0.0 0.0 0" rpy="0 0 0" />
+              <parent link="base_hub"/>
+              <child link="inertial_link_base_range_joint_${id}"/>
+            </joint>
             <gazebo reference="base_range_${id}">
                 <material>Gazebo/Yellow</material>
