Commit message: Add hub_id prefix to "base_hub" when multi-hub is enabled

File: urdf/base_hub.urdf.xacro (robot description, xacro)
@@ -19,5 +19,5 @@
           <joint name="hub_${hub_id}_gyro_joint" type="fixed">
               <origin xyz="0.0 0.0 0" rpy="0 0 -3.1415" />
-              <parent link="base_hub" />
+              <parent link="base_hub_${hub_id}" />
               <child link="hub_${hub_id}_gyro_link" />
           </joint>

Commit message: Update base_hub.urdf.xacro

File: urdf/base_hub.urdf.xacro (robot description, xacro)
@@ -24,7 +24,7 @@
           <link name="inertial_link_${hub_id}">
               <inertial>
-                  <mass value="0.3"/>
+                  <mass value="0.013"/>
                   <origin xyz="0 0 0"/>
-                  <cylinder_inertia m="0.1" r="0.6" h="0.03" />
+                  <cylinder_inertia m="0.013" r="0.06" h="0.03" />
               </inertial>
           </link>
@@ -64,5 +64,5 @@
                   <mass value="0.3"/>
                   <origin xyz="0 0 0"/>
-                  <cylinder_inertia m="0.1" r="0.6" h="0.03" />
+                  <cylinder_inertia m="0.013" r="0.06" h="0.03" />
               </inertial>
           </link>

Commit message: Correct mass value for single hub

File: urdf/base_hub.urdf.xacro (robot description, xacro)
@@ -62,5 +62,5 @@
           <link name="inertial_link">
               <inertial>
-                  <mass value="0.3"/>
+                  <mass value="0.013"/>
                   <origin xyz="0 0 0"/>
                   <cylinder_inertia m="0.013" r="0.06" h="0.03" />
